Commit message: minor changes to claw

File: urdf/claw.xacro (robot description, xacro)
@@ -7,5 +7,5 @@
     <inertial>
       <origin
-        xyz="-1.53567078563934E-16 1.27659406015648E-16 -0.0038047544848005"
+        xyz="-1.57328618926919E-16 1.27659406015648E-16 -0.00380475448480049"
         rpy="0 0 0" />
       <mass
@@ -13,8 +13,8 @@
       <inertia
         ixx="0.147608042754936"
-        ixy="4.79981990091153E-16"
-        ixz="-5.65036739485358E-17"
+        ixy="4.93667272888974E-16"
+        ixz="-6.23719916937828E-17"
         iyy="0.147608042754937"
-        iyz="2.48926524982492E-17"
+        iyz="1.15095319316312E-17"
         izz="0.226294089634963" />
     </inertial>
@@ -51,15 +51,15 @@
     <inertial>
       <origin
-        xyz="0.0390359916352672 -0.118859916128799 -2.77555756156289E-16"
-        rpy="0 0 0" />
-      <mass
-        value="5.8379618805716" />
-      <inertia
-        ixx="0.0430554980468734"
-        ixy="0.00387716715251265"
-        ixz="-5.20417042793042E-18"
-        iyy="0.00809595707264626"
-        iyz="2.53432257818487E-17"
-        izz="0.0494994685365442" />
+        xyz="0.05746 -0.11113 5.3429E-16"
+        rpy="0 0 0" />
+      <mass
+        value="5.838" />
+      <inertia
+        ixx="0.040951"
+        ixy="0.0091749"
+        ixz="-1.3878E-17"
+        iyy="0.010201"
+        iyz="6.6163E-17"
+        izz="0.049499" />
     </inertial>
     <visual>
@@ -74,5 +74,5 @@
         name="">
         <color
-          rgba="0.647058823529412 0.619607843137255 0.588235294117647 1" />
+          rgba="0.64706 0.61961 0.58824 1" />
       </material>
     </visual>
@@ -106,5 +106,5 @@
     <mimic
       joint="rod_joint"
-      multiplier="3"
+      multiplier="9.28356454545"
       offset="0" />
   </joint>
@@ -113,15 +113,15 @@
     <inertial>
       <origin
-        xyz="0.0390359916355864 -0.118859916128943 -2.44942954807925E-15"
-        rpy="0 0 0" />
-      <mass
-        value="5.8379618805716" />
-      <inertia
-        ixx="0.0430554980468635"
-        ixy="0.00387716715255743"
-        ixz="3.46944695195361E-18"
-        iyy="0.00809595707265621"
-        iyz="8.13151629364128E-18"
-        izz="0.0494994685365442" />
+        xyz="0.05746 -0.11113 -2.4286E-15"
+        rpy="0 0 0" />
+      <mass
+        value="5.838" />
+      <inertia
+        ixx="0.040951"
+        ixy="0.0091749"
+        ixz="-3.4694E-18"
+        iyy="0.010201"
+        iyz="1.4908E-17"
+        izz="0.049499" />
     </inertial>
     <visual>
@@ -136,5 +136,5 @@
         name="">
         <color
-          rgba="0.647058823529412 0.619607843137255 0.588235294117647 1" />
+          rgba="0.64706 0.61961 0.58824 1" />
       </material>
     </visual>
@@ -168,5 +168,5 @@
     <mimic
       joint="rod_joint"
-      multiplier="3"
+      multiplier="9.28356454545"
       offset="0" />
   </joint>
@@ -175,15 +175,15 @@
     <inertial>
       <origin
-        xyz="0.03903599163533 -0.11885991612886 -9.56495999594962E-18"
-        rpy="0 0 0" />
-      <mass
-        value="5.83796188057159" />
-      <inertia
-        ixx="0.0430554980468729"
-        ixy="0.00387716715251506"
-        ixz="4.88121916477368E-19"
-        iyy="0.00809595707264681"
-        iyz="1.26361575054972E-18"
-        izz="0.0494994685365442" />
+        xyz="0.05746 -0.11113 -7.0719E-18"
+        rpy="0 0 0" />
+      <mass
+        value="5.838" />
+      <inertia
+        ixx="0.040951"
+        ixy="0.0091749"
+        ixz="-3.6834E-19"
+        iyy="0.010201"
+        iyz="-2.2745E-19"
+        izz="0.049499" />
     </inertial>
     <visual>
@@ -198,5 +198,5 @@
         name="">
         <color
-          rgba="0.647058823529412 0.619607843137255 0.588235294117647 1" />
+          rgba="0.64706 0.61961 0.58824 1" />
       </material>
     </visual>
@@ -230,5 +230,5 @@
     <mimic
       joint="rod_joint"
-      multiplier="3"
+      multiplier="9.28356454545"
       offset="0" />
   </joint>
@@ -286,6 +286,6 @@
       xyz="0 1 0" />
     <limit
-      lower="0.05"
-      upper="-0.15"
+      lower="0.00"
+      upper="-0.11"
       effort="30"
       velocity="1" />
@@ -295,15 +295,15 @@
     <inertial>
       <origin
-        xyz="1.40630922126461E-15 0.0199999999998497 -6.57442263708274E-16"
-        rpy="0 0 0" />
-      <mass
-        value="3.66414183414919" />
-      <inertia
-        ixx="0.0072055452249317"
-        ixy="2.26087854114052E-19"
-        ixz="3.28399160889535E-17"
-        iyy="0.0134434480451304"
-        iyz="2.79163530569318E-19"
-        izz="0.00720554522493167" />
+        xyz="1.0298E-15 0.041745 -5.0073E-16"
+        rpy="0 0 0" />
+      <mass
+        value="3.4745" />
+      <inertia
+        ixx="0.0067165"
+        ixy="2.931E-19"
+        ixz="3.1841E-17"
+        iyy="0.012516"
+        iyz="2.2166E-19"
+        izz="0.0067165" />
     </inertial>
     <visual>
@@ -318,5 +318,5 @@
         name="">
         <color
-          rgba="0.647058823529412 0.619607843137255 0.588235294117647 1" />
+          rgba="0.64706 0.61961 0.58824 1" />
       </material>
     </visual>
@@ -335,5 +335,5 @@
     type="fixed">
     <origin
-      xyz="0 -0.10933 0"
+      xyz="0 -0.109328458561404 0"
       rpy="0 0 0" />
     <parent
@@ -348,15 +348,15 @@
     <inertial>
       <origin
-        xyz="0.016488 -0.031374 -0.021066"
+        xyz="0.015913 0.031888 0.020735"
         rpy="0 0 0" />
       <mass
         value="0.46607" />
       <inertia
-        ixx="0.00031785"
-        ixy="0.00015576"
-        ixz="6.9832E-05"
-        iyy="0.00019234"
-        iyz="-8.9929E-05"
-        izz="0.00039848" />
+        ixx="0.00032347"
+        ixy="-0.00015408"
+        ixz="-6.6582E-05"
+        iyy="0.00018484"
+        iyz="-8.8957E-05"
+        izz="0.00040036" />
     </inertial>
     <visual>
@@ -386,77 +386,85 @@
   <joint
     name="finger_a_support_joint"
-    type="fixed">
-    <origin
-      xyz="-0.081292 0.02 0.058481"
-      rpy="0 0 0" />
+    type="revolute">
+    <origin
+      xyz="-0.081292 0.041745 0.058481"
+      rpy="3.1416 0 0" />
     <parent
       link="moving_base" />
     <child
       link="finger_a_support" />
-    <axis
-      xyz="0.5 0 0.86603" />
-    <limit
-      lower="-3.14"
-      upper="1.5078"
-      effort="30"
-      velocity="1" />
-  </joint>
-  <link
-    name="finger_b_support">
-    <inertial>
-      <origin
-        xyz="0.0264880034316608 -0.0313744207600376 0.00374585052777678"
-        rpy="0 0 0" />
-      <mass
-        value="0.466065036871758" />
-      <inertia
-        ixx="0.000317845436466084"
-        ixy="0.000155761107485711"
-        ixz="-6.98321301226401E-05"
-        iyy="0.000192341398955658"
-        iyz="8.99287173361822E-05"
-        izz="0.000398480634714818" />
-    </inertial>
-    <visual>
-      <origin
-        xyz="0 0 0"
-        rpy="0 0 0" />
-      <geometry>
-        <mesh
-          filename="package://robots/meshes/claw/finger_b_support.STL" />
-      </geometry>
-      <material
-        name="">
-        <color
-          rgba="0.647058823529412 0.619607843137255 0.588235294117647 1" />
-      </material>
-    </visual>
-    <collision>
-      <origin
-        xyz="0 0 0"
-        rpy="0 0 0" />
-      <geometry>
-        <mesh
-          filename="package://robots/meshes/claw/finger_b_support.STL" />
-      </geometry>
-    </collision>
-  </link>
-  <joint
-    name="finger_b_support_joint"
-    type="fixed">
-    <origin
-      xyz="0.091292 0.02 0.04116"
-      rpy="-3.1416 0 3.1416" />
-    <parent
-      link="moving_base" />
-    <child
-      link="finger_b_support" />
     <axis
       xyz="0.5 0 -0.86603" />
     <limit
-      lower="-3.14"
-      upper="1.5078"
-      effort="30"
-      velocity="1" />
+      lower="-6.14"
+      upper="3.14"
+      effort="30"
+      velocity="1" />
+    <mimic
+      joint="rod_joint"
+      multiplier="12"
+      offset="0" />
+  </joint>
+  <link
+    name="finger_b_support">
+    <inertial>
+      <origin
+        xyz="0.025913 0.031888 -0.0034141"
+        rpy="0 0 0" />
+      <mass
+        value="0.46607" />
+      <inertia
+        ixx="0.00032347"
+        ixy="-0.00015408"
+        ixz="6.6582E-05"
+        iyy="0.00018484"
+        iyz="8.8957E-05"
+        izz="0.00040036" />
+    </inertial>
+    <visual>
+      <origin
+        xyz="0 0 0"
+        rpy="0 0 0" />
+      <geometry>
+        <mesh
+          filename="package://robots/meshes/claw/finger_b_support.STL" />
+      </geometry>
+      <material
+        name="">
+        <color
+          rgba="0.64706 0.61961 0.58824 1" />
+      </material>
+    </visual>
+    <collision>
+      <origin
+        xyz="0 0 0"
+        rpy="0 0 0" />
+      <geometry>
+        <mesh
+          filename="package://robots/meshes/claw/finger_b_support.STL" />
+      </geometry>
+    </collision>
+  </link>
+  <joint
+    name="finger_b_support_joint"
+    type="revolute">
+    <origin
+      xyz="0.091292 0.041745 0.04116"
+      rpy="0 0 -3.1416" />
+    <parent
+      link="moving_base" />
+    <child
+      link="finger_b_support" />
+    <axis
+      xyz="-0.5 0 -0.86603" />
+	<limit
+      lower="-6.14"
+      upper="6.14"
+      effort="30"
+      velocity="1" />
+      <mimic
+      joint="rod_joint"
+      multiplier="12"
+      offset="0" />
   </joint>
   <link
@@ -464,5 +472,5 @@
     <inertial>
       <origin
-        xyz="0.01 -0.031374 0.024812"
+        xyz="0.01 -0.031888 0.024149"
         rpy="0 0 0" />
       <mass
@@ -470,9 +478,9 @@
       <inertia
         ixx="0.0004388"
-        ixy="-1.3636E-21"
-        ixz="-1.4872E-21"
-        iyy="0.00019234"
-        iyz="0.00017986"
-        izz="0.00027753" />
+        ixy="-4.1141E-19"
+        ixz="3.1913E-19"
+        iyy="0.00018484"
+        iyz="0.00017791"
+        izz="0.00028503" />
     </inertial>
     <visual>
@@ -502,7 +510,7 @@
   <joint
     name="finger_c_support_joint"
-    type="fixed">
-    <origin
-      xyz="-0.01 0.02 -0.099641"
+    type="revolute">
+    <origin
+      xyz="-0.01 0.041745 -0.099641"
       rpy="0 0 0" />
     <parent
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